File: input_and_output_pins.kicad_sch (KiCad schematic)
At the start: 2 parts, among them J10 Screw_Terminal_01x03, J11 Screw_Terminal_01x03

Commit message: first schematic review
Other:
- note added: "just something small. common syntax in schematics is to have ground symbols pointing down and power rail sysmbols pointing up. doesn't affect anything, just looks better did it for you here, but just seomthing to keep in mind."
- moved on the sheet: J10
Changed lines of the file:
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@@
+		)
+	)
+	(text "just something small.\ncommon syntax in schematics is to have ground symbols pointing down\nand power rail sysmbols pointing up.\ndoesn't affect anything, just looks better\ndid it for you here, but just seomthing to keep in mind."
+		(exclude_from_sim no)
+		(at 102.108 24.638 0)
+		(effects
+			(font
+				(size 1.27 1.27)
+				(color 255 0 5 1)
+			)
 		)
 	)
@@
 				(size 1.27 1.27)
 			)
+		)
+	)
+	(wire
+		(pts
+			(xy 44.45 46.99) (xy 44.45 45.72)
+		)
+		(stroke
+			(width 0)
+			(type default)
 		)
 	)
@@
 	(global_label "Output_PWM"
 		(shape input)
-		(at 33.02 22.86 180)
+		(at 33.02 21.59 180)
 		(fields_autoplaced yes)
 		(effects
@@
 		)
 		(property "Intersheetrefs" "${INTERSHEET_REFS}"
-			(at 18.6655 22.86 0)
+			(at 18.6655 21.59 0)
 			(hide yes)
 			(show_name no)
@@
 	(global_label "Output_VCC"
 		(shape input)
-		(at 33.02 25.4 180)
+		(at 33.02 24.13 180)
 		(fields_autoplaced yes)
 		(effects
@@
 		)
 		(property "Intersheetrefs" "${INTERSHEET_REFS}"
-			(at 19.2097 25.4 0)
+			(at 19.2097 24.13 0)
 			(hide yes)
 			(show_name no)
@@
 		(polyline
 			(pts
-				(xy 17.78 36.83) (xy 76.2 36.83) (xy 76.2 49.53) (xy 17.78 49.53)
+				(xy 17.78 36.83) (xy 76.2 36.83) (xy 76.2 53.34) (xy 17.78 53.34)
 			)
 			(stroke
@@
 	(symbol
 		(lib_id "power:GND")
-		(at 44.45 45.72 270)
+		(at 44.45 46.99 0)
 		(unit 1)
 		(body_style 1)
@@
 		(in_pos_files yes)
 		(dnp no)
-		(fields_autoplaced yes)
 		(property "Reference" "#PWR051"
-			(at 38.1 45.72 0)
+			(at 44.45 53.34 0)
 			(hide yes)
 			(show_name no)
@@
 		)
 		(property "Value" "GND"
-			(at 40.64 45.7199 90)
-			(show_name no)
-			(do_not_autoplace no)
-			(effects
-				(font
-					(size 1.27 1.27)
-				)
-				(justify right)
+			(at 42.672 50.8 0)
+			(show_name no)
+			(do_not_autoplace no)
+			(effects
+				(font
+					(size 1.27 1.27)
+				)
+				(justify left)
 			)
 		)
 		(property "Footprint" ""
-			(at 44.45 45.72 0)
+			(at 44.45 46.99 0)
 			(hide yes)
 			(show_name no)
@@
 		)
 		(property "Datasheet" ""
-			(at 44.45 45.72 0)
+			(at 44.45 46.99 0)
 			(hide yes)
 			(show_name no)
@@
 		)
 		(property "Description" "Power symbol creates a global label with name \"GND\" , ground"
-			(at 44.45 45.72 0)
+			(at 44.45 46.99 0)
 			(hide yes)
 			(show_name no)
@@
 	(symbol
 		(lib_id "Connector:Screw_Terminal_01x03")
-		(at 38.1 25.4 0)
+		(at 38.1 24.13 0)
 		(unit 1)
 		(body_style 1)
@@
 		(fields_autoplaced yes)
 		(property "Reference" "J10"
-			(at 40.64 24.1299 0)
+			(at 40.64 22.8599 0)
 			(show_name no)
 			(do_not_autoplace no)
@@
 		)
 		(property "Value" "Screw_Terminal_01x03"
-			(at 40.64 26.6699 0)
+			(at 40.64 25.3999 0)
 			(show_name no)
 			(do_not_autoplace no)
@@
 		)
 		(property "Footprint" ""
-			(at 38.1 25.4 0)
+			(at 38.1 24.13 0)
 			(hide yes)
 			(show_name no)
@@
 		)
 		(property "Datasheet" ""
-			(at 38.1 25.4 0)
+			(at 38.1 24.13 0)
 			(hide yes)
 			(show_name no)
@@
 		)
 		(property "Description" "Generic screw terminal, single row, 01x03, script generated (kicad-library-utils/schlib/autogen/connector/)"
-			(at 38.1 25.4 0)
+			(at 38.1 24.13 0)
 			(hide yes)
 			(show_name no)
@@
 	(symbol
 		(lib_id "power:GND")
-		(at 33.02 27.94 270)
+		(at 33.02 26.67 0)
 		(unit 1)
 		(body_style 1)
@@
 		(in_pos_files yes)
 		(dnp no)
-		(fields_autoplaced yes)
 		(property "Reference" "#PWR050"
-			(at 26.67 27.94 0)
+			(at 33.02 33.02 0)
 			(hide yes)
 			(show_name no)
@@
 		)
 		(property "Value" "GND"
-			(at 29.21 27.9399 90)
-			(show_name no)
-			(do_not_autoplace no)
-			(effects
-				(font
-					(size 1.27 1.27)
-				)
-				(justify right)
+			(at 30.988 30.48 0)
+			(show_name no)
+			(do_not_autoplace no)
+			(effects
+				(font
+					(size 1.27 1.27)
+				)
+				(justify left)
 			)
 		)
 		(property "Footprint" ""
-			(at 33.02 27.94 0)
+			(at 33.02 26.67 0)
 			(hide yes)
 			(show_name no)
@@
 		)
 		(property "Datasheet" ""
-			(at 33.02 27.94 0)
+			(at 33.02 26.67 0)
 			(hide yes)
 			(show_name no)
@@
 		)
 		(property "Description" "Power symbol creates a global label with name \"GND\" , ground"
-			(at 33.02 27.94 0)
-			(hide yes)
-			(show_name no)
+			(at 33.02 26.67 0)
+			(hide yes)
+			(show_name no)

Commit message: Add files via upload
Revisions V2
Other:
- note removed: "just something small. common syntax in schematics is to have ground symbols pointing down and power rail sysmbols pointing up. doesn't affect anything, just looks better did it for you here, but just seomthing to keep in mind."
Changed lines of the file:
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@@
-		)
-	)
-	(text "just something small.\ncommon syntax in schematics is to have ground symbols pointing down\nand power rail sysmbols pointing up.\ndoesn't affect anything, just looks better\ndid it for you here, but just seomthing to keep in mind."
-		(exclude_from_sim no)
-		(at 102.108 24.638 0)
-		(effects
-			(font
-				(size 1.27 1.27)
-				(color 255 0 5 1)
-			)
 		)
 	)
