File: Airbrake Redundancy Board.kicad_sch (KiCad schematic)
At the start: 20 parts, among them J5 USB_C_Receptacle_USB2.0_16P, SW3 SW_Push, SW4 SW_Push, U1 TPD1E05U06DPY, U6 RT9080-33GJ5, U7 ESP32-C3-WROOM-02

Commit message: first schematic review
Other:
- note added: "Add ESD protection for the data lines"
- note added: "add decoupling caps here. general rule to have caps on power lines"
- note added: "dont need esd protection here. only need esd protection for outside connections. for example, your data line connections need it, but your 3.3V orginating from your own LDO doesn't"
- note added: "double check me, but i dont think you can use io6 for adc reading"
- note added: "make sure youre accounting for the drop across this diode. like, ensure youre 5V line is ok with being a little lower than 5V. I see the jumper but then that kinda eliminates the whole point, no?"
- note added: "this symbol isn't matching what I see on the datasheet. the BP pin is showing as SNS. looking into it, seems like that datasheet and this symbol are two different ICs. double check which one you want to run with, and clarify"
Changed lines of the file:
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@@
 		(company "LRA")
+	)
+	(text "Add ESD protection for the data lines"
+		(exclude_from_sim no)
+		(at 53.086 48.514 0)
+		(effects
+			(font
+				(size 1.27 1.27)
+				(color 255 0 5 1)
+			)
+		)
+	)
+	(text "double check me, but i dont think you can use io6 for adc reading"
+		(exclude_from_sim no)
+		(at 179.832 66.294 0)
+		(effects
+			(font
+				(size 1.27 1.27)
+				(color 255 0 5 1)
+			)
+		)
+	)
+	(text "make sure youre accounting for the drop across this diode.\nlike, ensure youre 5V line is ok with being a little lower than 5V.\nI see the jumper but then that kinda eliminates the whole point, no?"
+		(exclude_from_sim no)
+		(at 43.942 91.948 0)
+		(effects
+			(font
+				(size 1.27 1.27)
+				(color 255 0 5 1)
+			)
+		)
 	)
 	(text "USBC Power Regulator"
@@
 			)
 		)
+	)
+	(text "dont need esd protection here. \nonly need esd protection for outside connections.\nfor example, your data line connections need it, but your 3.3V\norginating from your own LDO doesn't"
+		(exclude_from_sim no)
+		(at 164.084 123.952 0)
+		(effects
+			(font
+				(size 1.27 1.27)
+				(color 255 0 5 1)
+			)
+		)
+	)
+	(text "add decoupling caps here.\ngeneral rule to have caps on power lines"
+		(exclude_from_sim no)
+		(at 48.514 23.368 0)
+		(effects
+			(font
+				(size 1.27 1.27)
+				(color 255 0 5 1)
+			)
+		)
+	)
+	(text "this symbol isn't matching what I see on the datasheet.\nthe BP pin is showing as SNS.\nlooking into it, seems like that datasheet and this symbol are two\ndifferent ICs.\n\ndouble check which one you want to run with, and clarify\n"
+		(exclude_from_sim no)
+		(at 44.196 144.018 0)
+		(effects
+			(font
+				(size 1.27 1.27)
+				(color 255 0 5 1)
+			)
+		)

Commit message: Add files via upload
Revisions V2
Parts:
- removed U6: RT9080-33GJ5, Package_TO_SOT_SMD:SOT-23-5, symbol Regulator_Linear:AP131-33
- added C1: 10 μF, symbol Device:C_Small_US
- added U3: TPD1E05U06DPY, Package_SON:Texas_DPY0002A_0.6x1mm_P0.65mm, symbol Power_Protection:TPD1E05U06DPY
- added U4: TLV70033_SOT23-5, Package_TO_SOT_SMD:SOT-23-5, symbol Regulator_Linear:TLV70033_SOT23-5
Connections:
- net IO4 is gone; now on net Main Board VCC Step Down: U7.3 (GPIO4/ADC1_CH4)
- net +3V3: no longer U1.1 (I/O)
- net +5V: now also U4.1 (IN), U4.3 (EN)
- net GND: now also C1.2, U3.2 (GND), U4.2 (GND)
- net IO18: now also U3.1 (I/O)
- net IO19: now also U1.1 (I/O)
- net Main Board VCC Step Down: no longer U7.5 (GPIO6)
- net VBUS: now also C1.1
- net at C6.1, JP4.1 (A): now also U4.5 (OUT)
- new net IO6: U7.5 (GPIO6)
Other:
- note added: "Changed to protect data lines from USBC"
- note added: "I changed the IC entirely. It says it's rated for 200 mA and im not entirely sure how to ensure that the ESP32 isn't drawing more than that so if pls lemme know if itll work"
- note added: "added decoupling cap I lowkey don't know how to calculate value so this needs to be double checked"
- note added: "changed from io6 to io4 because of ADC compatibility"
- note added: "voltage drop across the diode is 0.6V so that would make the +5V be 4.4V. The TLV70033 below has an operating input voltage of -0.3V to 6V so it should be chill"
- note removed: "Add ESD protection for the data lines"
- note removed: "add decoupling caps here. general rule to have caps on power lines"
- note removed: "dont need esd protection here. only need esd protection for outside connections. for example, your data line connections need it, but your 3.3V orginating from your own LDO doesn't"
- note removed: "double check me, but i dont think you can use io6 for adc reading"
- note removed: "make sure youre accounting for the drop across this diode. like, ensure youre 5V line is ok with being a little lower than 5V. I see the jumper but then that kinda eliminates the whole point, no?"
- note removed: "this symbol isn't matching what I see on the datasheet. the BP pin is showing as SNS. looking into it, seems like that datasheet and this symbol are two different ICs. double check which one you want to run with, and clarify"

Commit message: second review
Other:
- note added: "THE ESP32's datasheet usually has a current load amount somewhere. I would make sure this LDO can handle the MAX the ESP pulls. ik that the wifi chips on ESP's are quite load intensive. I would personally just go through and calculate how much current you expect to be pulled. if it is low enough (for this 200mA limit), stick with this LDO. if not, switch it out. safe bet is to juse assume the ESP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"
- note added: "i would stick with non polarized caps for your application."
- note removed: "Changed to protect data lines from USBC"
- note removed: "I changed the IC entirely. It says it's rated for 200 mA and im not entirely sure how to ensure that the ESP32 isn't drawing more than that so if pls lemme know if itll work"
- note removed: "added decoupling cap I lowkey don't know how to calculate value so this needs to be double checked"
- note removed: "changed from io6 to io4 because of ADC compatibility"
- note removed: "voltage drop across the diode is 0.6V so that would make the +5V be 4.4V. The TLV70033 below has an operating input voltage of -0.3V to 6V so it should be chill"
Changed lines of the file:
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@@
 		(company "LRA")
-	)
-	(text "changed from io6 to io4 because of ADC compatibility"
-		(exclude_from_sim no)
-		(at 173.99 61.214 0)
-		(effects
-			(font
-				(size 1.27 1.27)
-				(color 255 0 5 1)
-			)
-		)
-	)
-	(text "voltage drop across the diode is 0.6V \nso that would make the +5V be 4.4V.\nThe TLV70033 below has an operating\n input voltage of -0.3V to 6V so it should be chill"
-		(exclude_from_sim no)
-		(at 43.942 92.964 0)
-		(effects
-			(font
-				(size 1.27 1.27)
-				(color 255 0 5 1)
-			)
-		)
 	)
 	(text "USBC Power Regulator"
@@
 			(font
 				(size 1.27 1.27)
-			)
-		)
-	)
-	(text "Changed to protect data lines from USBC"
-		(exclude_from_sim no)
-		(at 176.022 102.87 0)
-		(effects
-			(font
-				(size 1.27 1.27)
-				(color 242 0 0 1)
 			)
 		)
@@
 		)
 	)
-	(text "added decoupling cap\nI lowkey don't know how to calculate value\n so this needs to be double checked"
+	(text "i would stick with non polarized caps for your application."
 		(exclude_from_sim no)
 		(at 64.77 21.336 0)
@@
 		)
 	)
-	(text "I changed the IC entirely. It says it's\nrated for 200 mA and im not entirely sure\nhow to ensure that the ESP32 isn't drawing more\nthan that so if pls lemme know if itll work"
+	(text "THE ESP32's datasheet usually has a current load amount somewhere.\nI would make sure this LDO can handle the MAX the ESP pulls.\nik that the wifi chips on ESP's are quite load intensive.\nI would personally just go through and calculate how much current you\nexpect to be pulled. if it is low enough (for this 200mA limit),\nstick with this LDO. if not, switch it out.\n\nsafe bet is to juse assume the ESP will pull the max current it states\nin its sheet and using that as a constraint for which LDO you run with."
 		(exclude_from_sim no)
-		(at 39.878 152.654 0)
+		(at 46.99 157.988 0)
 		(effects
 			(font
