File: pwm_management.kicad_sch (KiCad schematic)
At the start: 4 parts, among them Q5 AO3401A, Q6 DMN30H4D0L, Q7 AO3401A, Q8 DMN30H4D0L

Commit message: first schematic review
Other:
- note added: "look into how youre supposed to configure a pmos circuit. currently if you ran with this, when the nmos is off, the pmos would be 'floating' causing issues. you need to add a pull up resistor of soem sort, like i did in my circuit. also i highly suggest adding pull down resistors to youre nmos gates to ensure that when you make them low, they 'actually' become low. it just a way to ensure the lin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"
Changed lines of the file:
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@@
+		)
+	)
+	(text "look into how youre supposed to configure a pmos circuit.\ncurrently if you ran with this, when the nmos is off, the pmos\nwould be 'floating' causing issues.\n\nyou need to add a pull up resistor of soem sort, like i did in my\ncircuit.\n\nalso i highly suggest adding pull down resistors to youre nmos gates to ensure\nthat when you make them low, they 'actually' become low.\nit just a way to ensure the line actually hits 0V.\n\nalso add gate resistors for the nmos to protect the ic."
+		(exclude_from_sim no)
+		(at 78.232 72.898 0)
+		(effects
+			(font
+				(size 1.27 1.27)
+				(color 255 0 23 1)
+			)
 		)
 	)
@@
 	(symbol
 		(lib_id "power:GND")
-		(at 107.95 38.1 90)
+		(at 107.95 38.1 0)
 		(unit 1)
 		(body_style 1)
@@
 		(fields_autoplaced yes)
 		(property "Reference" "#PWR053"
-			(at 114.3 38.1 0)
+			(at 107.95 44.45 0)
 			(hide yes)
 			(show_name no)
@@
 		)
 		(property "Value" "GND"
-			(at 113.03 38.1 0)
-			(show_name no)
-			(do_not_autoplace no)
-			(effects
-				(font
-					(size 1.27 1.27)
-				)
+			(at 110.49 39.3699 0)
+			(show_name no)
+			(do_not_autoplace no)
+			(effects
+				(font
+					(size 1.27 1.27)
+				)
+				(justify left)
 			)
 		)
@@
 	(symbol
 		(lib_id "power:GND")
-		(at 58.42 38.1 90)
+		(at 58.42 38.1 0)
 		(unit 1)
 		(body_style 1)
@@
 		(fields_autoplaced yes)
 		(property "Reference" "#PWR046"
-			(at 64.77 38.1 0)
+			(at 58.42 44.45 0)
 			(hide yes)
 			(show_name no)
@@
 		)
 		(property "Value" "GND"
-			(at 63.5 38.1 0)
-			(show_name no)
-			(do_not_autoplace no)
-			(effects
-				(font
-					(size 1.27 1.27)
-				)
-			)
-		)
+			(at 60.96 39.3699 0)
+			(show_name no)
+			(do_not_autoplace no)
+			(effects
+				(font
+					(size 1.27 1.27)
+				)
+				(justify left)
+			)
+		)

Commit message: Add files via upload
Revisions V2
Parts:
- added R16, R17: 1k Ω, symbol Device:R_US
- added R3, R4, R5, R6: 10k Ω, symbol Device:R_US
Connections:
- net 1OE: now also R16.2; no longer Q6.1 (G)
- net 2OE: now also R17.2; no longer Q8.1 (G)
- net GND: now also R3.1, R5.1
- net at Q7.1 (G), Q8.2 (S): now also R6.2
- net at Q5.1 (G), Q6.2 (S): now also R4.2
- new net: Q6.1 (G), R16.1, R3.2
- new net: Q8.1 (G), R17.1, R5.2
- new net +3V3: R4.1, R6.1
Other:
- note added: "added pull up, pull down, and gate resistors. I think 10k for both the pull up and down resistors should be enough but i hand waved that. Same thing with the 1k gate resistor"
- note removed: "look into how youre supposed to configure a pmos circuit. currently if you ran with this, when the nmos is off, the pmos would be 'floating' causing issues. you need to add a pull up resistor of soem sort, like i did in my circuit. also i highly suggest adding pull down resistors to youre nmos gates to ensure that when you make them low, they 'actually' become low. it just a way to ensure the lin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"

Commit message: second review
Other:
- note added: "i think the nmos might be backwards, double check. current flows drain to source for an nmos also double check that the gate voltgae will ALWAYS be higher than the pwm signal to ensure it actually turns off. I also asked another friend about this and he said that it might be smart to put another pmos, like source to source, to prevent leakage incase the pmos does not turn fully off. look more int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"
- note removed: "added pull up, pull down, and gate resistors. I think 10k for both the pull up and down resistors should be enough but i hand waved that. Same thing with the 1k gate resistor"
Changed lines of the file:
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@@
 		)
 	)
-	(text "added pull up, pull down, and gate resistors.\n I think 10k for both the pull up and down resistors\nshould be enough but i hand waved that. Same thing\nwith the 1k gate resistor"
+	(text "i think the nmos might be backwards, double check.\ncurrent flows drain to source for an nmos\n\nalso double check that the gate voltgae will ALWAYS be higher than the \npwm signal to ensure it actually turns off.\n\nI also asked another friend about this and he said that it might\nbe smart to put another pmos, like source to source, to prevent\nleakage incase the pmos does not turn fully off. look more into that\nroute.\nthis lowkey caused me to think more about this and it might be\nsmarter to use some sort of MUX system instead of this, as I forgot\nthe PWM signal is very delicate. if old PWM accidently starts to combine\nwith the new PWM, it could cause BIG issues with the servo. look into\nthis route as well and see if you agree with me or not.\n\nalso add a pull down on the output pwm to ensure it clears the line\nwhen the switch does happen."
 		(exclude_from_sim no)
-		(at 73.152 65.532 0)
+		(at 73.406 78.994 0)
 		(effects
 			(font
