File: vcc_management.kicad_sch (KiCad schematic)
At the start: 8 parts, among them J1 Screw_Terminal_01x02, Q10 DMN30H4D0L, Q11 AO3401A, Q12 DMN30H4D0L, Q9 AO3401A, U2 AZ1117CH2-5.0

Commit message: first schematic review
Other:
- note added: "actually put values for resistors here. otherwise i cannot check if this voltage divider will work or not"
- note added: "double check me, but i dont think you can use io6 for adc reading"
- note added: "look in the datasheet to see how they hook up the IC. youre not using any of the passives they want to be used. this circuit may not work as inteded then."
- note added: "same issues with the pwm_managment high side circuit"
Changed lines of the file:
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@@
+		)
+	)
+	(text "look in the datasheet to see how they hook up the IC.\nyoure not using any of the passives they want to be used.\nthis circuit may not work as inteded then."
+		(exclude_from_sim no)
+		(at 44.45 157.734 0)
+		(effects
+			(font
+				(size 1.27 1.27)
+				(color 255 0 5 1)
+			)
+		)
+	)
+	(text "same issues with the pwm_managment high side circuit"
+		(exclude_from_sim no)
+		(at 143.002 56.388 0)
+		(effects
+			(font
+				(size 1.27 1.27)
+				(color 255 0 23 1)
+			)
 		)
 	)
@@
 			(font
 				(size 1.27 1.27)
+			)
+		)
+	)
+	(text "actually put values for resistors here.\notherwise i cannot check if this voltage divider will work\nor not"
+		(exclude_from_sim no)
+		(at 91.694 111.506 0)
+		(effects
+			(font
+				(size 1.27 1.27)
+				(color 255 0 5 1)
+			)
+		)
+	)
+	(text "double check me, but i dont think you can use io6 for adc reading"
+		(exclude_from_sim no)
+		(at 78.232 103.124 0)
+		(effects
+			(font
+				(size 1.27 1.27)
+				(color 255 0 5 1)
 			)
 		)
@@
 	(symbol
 		(lib_id "power:GND")
-		(at 53.34 116.84 90)
+		(at 53.34 116.84 0)
 		(unit 1)
 		(body_style 1)
@@
 		(dnp no)
 		(property "Reference" "#PWR052"
-			(at 59.69 116.84 0)
+			(at 53.34 123.19 0)
 			(hide yes)
 			(show_name no)
@@
 		)
 		(property "Value" "GND"
-			(at 58.42 116.84 90)
+			(at 53.594 120.65 0)
 			(show_name no)
 			(do_not_autoplace no)
@@
 	(symbol
 		(lib_id "power:GND")
-		(at 100.33 54.61 90)
+		(at 100.33 54.61 0)
 		(unit 1)
 		(body_style 1)
@@
 		(fields_autoplaced yes)
 		(property "Reference" "#PWR043"
-			(at 106.68 54.61 0)
+			(at 100.33 60.96 0)
 			(hide yes)
 			(show_name no)
@@
 		)
 		(property "Value" "GND"
-			(at 105.41 54.61 0)
-			(show_name no)
-			(do_not_autoplace no)
-			(effects
-				(font
-					(size 1.27 1.27)
-				)
+			(at 102.87 55.8799 0)
+			(show_name no)
+			(do_not_autoplace no)
+			(effects
+				(font
+					(size 1.27 1.27)
+				)
+				(justify left)
 			)
 		)
@@
 	(symbol
 		(lib_id "power:GND")
-		(at 50.8 54.61 90)
+		(at 50.8 54.61 0)
 		(unit 1)
 		(body_style 1)
@@
 		(fields_autoplaced yes)
 		(property "Reference" "#PWR042"
-			(at 57.15 54.61 0)
+			(at 50.8 60.96 0)
 			(hide yes)
 			(show_name no)
@@
 		)
 		(property "Value" "GND"
-			(at 55.88 54.61 0)
-			(show_name no)
-			(do_not_autoplace no)
-			(effects
-				(font
-					(size 1.27 1.27)
-				)
-			)
-		)
+			(at 53.34 55.8799 0)
+			(show_name no)
+			(do_not_autoplace no)
+			(effects
+				(font
+					(size 1.27 1.27)
+				)
+				(justify left)
+			)
+		)

Commit message: Add files via upload
Revisions V2
Parts:
- added C2: 10 µF, symbol Device:C_Small_US
- added C3: 22 µF, symbol Device:C_Small_US
- added R13, R14, R15, R7: 10k Ω, symbol Device:R_US
- added R18, R19: 1k Ω, symbol Device:R_US
- R1: value R_US -> 14.3k
- R2: value R_US -> 10k
Connections:
- net 1OE: now also R18.2; no longer Q10.1 (G)
- net 2OE: now also R19.2; no longer Q12.1 (G)
- net Back Up VCC: now also J1.1 (Pin_1), C2.1; no longer J1.2 (Pin_2)
- net GND: now also J1.2 (Pin_2), C2.2, C3.2, R13.1, R15.1; no longer J1.1 (Pin_1)
- net VBUS: now also C3.1
- net at Q11.1 (G), Q12.2 (S): now also R7.2
- net at Q10.2 (S), Q9.1 (G): now also R14.2
- new net: Q12.1 (G), R13.2, R19.1
- new net: Q10.1 (G), R15.2, R18.1
- new net +3V3: R14.1, R7.1
Other:
- note added: "Added a pull up, pull down, and gate resistor. Same hand wavey calcs for the gate resistors."
- note added: "i updated with the passives. I used the AZ1117C-3.3 for reference on page 3 (typical applications circuits)"
- note added: "voltage divider values put in for a stepdown from 8V to 3.3V"
- note removed: "actually put values for resistors here. otherwise i cannot check if this voltage divider will work or not"
- note removed: "double check me, but i dont think you can use io6 for adc reading"
- note removed: "look in the datasheet to see how they hook up the IC. youre not using any of the passives they want to be used. this circuit may not work as inteded then."
- note removed: "same issues with the pwm_managment high side circuit"

Commit message: second review
Other:
- note added: "again, stick to non polarized caps here if you are powering VBUS, you must ensure you NEVER have the battery pack for Bakc Up VCC and your USBC connected at the same time. currently you have two sources powering VBUS, keep this in mind. also, is Back UP VCC 8V? If so, I would look into a buck converter. 3V drop with an LDO will create A LOT of heat, could burn an IC."
- note added: "same thing about the nmos and pmos from other sheet. double check orientation and if the PMOS gate voltage is enough. add pull down on output line the whole leakage and sensative PWM signal stuff does not apply here. we can keep this as is, as we do not really care about a square wave in this scenario. also is input VCC expected to be 8V here? if so, the PMOS will not wotk with a 3.3V gate voltag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"
- note removed: "Added a pull up, pull down, and gate resistor. Same hand wavey calcs for the gate resistors."
- note removed: "i updated with the passives. I used the AZ1117C-3.3 for reference on page 3 (typical applications circuits)"
Changed lines of the file:
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@@
 		)
 	)
-	(text "i updated with the passives. \nI used the AZ1117C-3.3 for reference on page 3 (typical applications circuits)"
+	(text "again, stick to non polarized caps here\n\nif you are powering VBUS, you must ensure you NEVER have the battery pack\nfor Bakc Up VCC and your USBC connected at the same time. \ncurrently you have two sources powering VBUS, keep this in mind.\n\nalso, is Back UP VCC 8V? If so, I would look into a buck converter.\n3V drop with an LDO will create A LOT of heat, could burn an IC."
 		(exclude_from_sim no)
-		(at 54.102 157.226 0)
+		(at 54.102 163.322 0)
 		(effects
 			(font
@@
 		)
 	)
-	(text "Added a pull up, pull down, and gate resistor. \nSame hand wavey calcs for the gate resistors."
+	(text "same thing about the nmos and pmos from other sheet. double check orientation\nand if the PMOS gate voltage is enough. add pull down on output line\n\nthe whole leakage and sensative PWM signal stuff does not\napply here. we can keep this as is, as we do not really care about\na square wave in this scenario.\n\nalso is input VCC expected to be 8V here? if so,\nthe PMOS will not wotk with a 3.3V gate voltage."
 		(exclude_from_sim no)
-		(at 137.668 56.896 0)
+		(at 156.718 59.436 0)
 		(effects
 			(font
